File: Schematics/DMB-4770-8-IN-8-OUT.brd (EAGLE design)
At the start: 32.8 x 86.9 mm, 41 parts

Commit message: Modifications et ajout des cartes C
Parts:
- renumbered E$1 to J1, E$10 to R13, E$11 to R12, E$12 to R16, E$13 to R17, E$14 to R18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
