File: Schematics/BeagleBrasse_cape.brd (EAGLE design)
At the start: 86.4 x 54.6 mm, 11 parts

Commit message: Ajout 1-wire
Parts:
- added E$5: (no value), connectors:JP03N
- added E$6: 4.7K, ref-packages:C0805
Connections:
- new net S$12: E$5.2, E$6.2, U$1.P9.25
- net S$17: now also E$5.1
- net S$19: now also E$5.3, E$6.1
Routing:
- net S$12: track 0.00 -> 34.3 mm
- net S$17: track 169.7 -> 191.5 mm
- net S$19: track 170.3 -> 184.2 mm
- net S$6: track 71.5 -> 70.4 mm

Commit message: Renomage
Routing:
- net S$18: track 43.1 -> 45.6 mm
Changed lines of the file:
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@@
 <contactref element="U$1" pad="P9.31"/>
 <wire x1="14.9225" y1="26.67" x2="14.9225" y2="46.355" width="0.4064" layer="1"/>
-<wire x1="27.94" y1="52.705" x2="26.67" y2="51.435" width="0.4064" layer="1"/>
-<wire x1="26.67" y1="51.435" x2="26.67" y2="48.26" width="0.4064" layer="1"/>
-<wire x1="26.67" y1="48.26" x2="25.7175" y2="47.3075" width="0.4064" layer="1"/>
-<wire x1="25.7175" y1="47.3075" x2="15.875" y2="47.3075" width="0.4064" layer="1"/>
+<wire x1="27.94" y1="52.705" x2="29.21" y2="51.435" width="0.4064" layer="1"/>
+<wire x1="29.21" y1="51.435" x2="29.21" y2="48.26" width="0.4064" layer="1"/>
+<wire x1="29.21" y1="48.26" x2="28.2575" y2="47.3075" width="0.4064" layer="1"/>
+<wire x1="28.2575" y1="47.3075" x2="15.875" y2="47.3075" width="0.4064" layer="1"/>
 <wire x1="15.875" y1="47.3075" x2="14.9225" y2="46.355" width="0.4064" layer="1"/>
 <wire x1="11.1125" y1="26.035" x2="14.2875" y2="26.035" width="0.4064" layer="1"/>
