File: Schematics/0 - I2C 2018/Pi Board.sch (EAGLE design)
At the start: 12 parts, among them J1 RASPBERRYPI-40-PIN-GPIO, U1 P82B715TD, X1 RJ45-8X, X2 RJ45-8X, X3 RJ45-8X, X4 RJ45-8X, X5 MKDSN1,5/2-5,08

Commit message: Finalisation interface PI
Parts:
- added C2, C3: (no value), resistor:CPOL-USC
- added U2: 7805T, linear:7805T
Connections:
- removed net +12V: R9.2, X5-2.KL
- removed net EXT_INT: X1.5, X2.5, X3.5, X4.5
- new net +5V: C3.+, J1.5V@2, J1.5V@4, U2.VO
- new net INT_1: J1.GP17, X1.5
- new net INT_2: J1.GP18#, X2.5
- new net INT_3: J1.GP27, X3.5
- new net INT_4: J1.GP25, X4.5
- net +12VBUS: now also C2.+, R9.2, U2.VI, X5-2.KL
- net DGND: now also C2.-, C3.-, U2.GND
